Commit message: Add UAV pose control and OMY F3M simulation

File: ros2_ws/src/uav_description/urdf/uav_ver62.urdf (robot description, URDF)
Before this commit: robot uav_ver62, 3 links, 2 joints
Links:
- link base_link: geometry collision mesh filename=../meshes/base_link.stl scale=0.0003 0.0003 0.0003; visual cylinder length=0.8 radius=0.025
- link left_wing_1: geometry collision mesh filename=../meshes/left_wing_1.stl scale=0.0003 0.0003 0.0003; visual mesh filename=../meshes/left_wing_1.stl scale=0.0003 0.0003 0.0003
- link right_wing_1: geometry collision mesh filename=../meshes/right_wing_1.stl scale=0.0003 0.0003 0.0003; visual mesh filename=../meshes/right_wing_1.stl scale=0.0003 0.0003 0.0003
Joints:
- joint joint_left_wing: origin xyz=0.075 -0.06 0.18 rpy=0 0 0 -> xyz=-0.075 0.06 0.18 rpy=0 0 3.141592653589793
- joint joint_right_wing: origin xyz=0.075 0.06 0.18 rpy=0 0 0 -> xyz=-0.075 -0.06 0.18 rpy=0 0 3.141592653589793
